Commit message: compatible with dave uuv simulator

File: bluerov2_description/robots/bluerov2_default_original.xacro (robot description, xacro)
@@ -3,6 +3,4 @@
   <xacro:arg name="debug" default="0"/>
   <xacro:arg name="namespace" default="bluerov2"/>
-  <!-- add this into file -->
-  <!-- <xacro:arg name="inertial_reference_frame" default="world"/> -->
   <!-- Include the ROV macro file xacro:bluerov2_base -->
   <xacro:include filename="$(find bluerov2_description)/urdf/base.xacro"/>
@@ -11,5 +9,4 @@
 <!-- Create the bluerov2 -->
   <xacro:bluerov2_base namespace="$(arg namespace)">
- <!--  inertial_reference_frame="$(arg inertial_reference_frame)" -->
     <!-- The underwater object plugin is given as an input block parameter to
      allow the addition of external models of manipulator units -->

File: bluerov2_description/robots/bluerov2_rlearning.xacro (robot description, xacro)
@@ -3,6 +3,4 @@
   <xacro:arg name="debug" default="0"/>
   <xacro:arg name="namespace" default="bluerov2"/>
-  <!-- add this into file -->
-  <!-- <xacro:arg name="inertial_reference_frame" default="world"/> -->
   <!-- Include the ROV macro file xacro:bluerov2_base -->
   <xacro:include filename="$(find bluerov2_description)/urdf/base.xacro"/>
@@ -11,5 +9,4 @@
 <!-- Create the bluerov2 -->
   <xacro:bluerov2_base namespace="$(arg namespace)">
- <!--  inertial_reference_frame="$(arg inertial_reference_frame)" -->
     <!-- The underwater object plugin is given as an input block parameter to
      allow the addition of external models of manipulator units -->
@@ -33,5 +30,3 @@
   <!-- Joint state publisher plugin -->
   <xacro:default_joint_state_publisher namespace="$(arg namespace)" update_rate="10"/>
-  <!-- Mount a Pose 3D sensor. -->
-  <xacro:default_pose_3d namespace="bluerov2" parent_link="bluerov2/base_link" />
 </robot>

File: bluerov2_description/urdf/base_backup.xacro (robot description, xacro)
@@ -21,9 +21,9 @@
   <!-- Volume -->
   <!-- <xacro:property name="volume" value="0.011054"/> -->
-  <xacro:property name="mass" value="26.75"/>
-  <xacro:property name="x_size" value="0.457"/>
-  <xacro:property name="y_size" value="0.338"/>
-  <xacro:property name="z_size" value="0.254"/>
-  <xacro:property name="volume" value="0.0261"/>
+  <xacro:property name="mass" value="20.5"/>
+  <xacro:property name="x_size" value="0.45"/>
+  <xacro:property name="y_size" value="0.35"/>
+  <xacro:property name="z_size" value="0.35"/>
+  <xacro:property name="volume" value="0.02"/>
   <!-- Center of gravity -->
   <xacro:property name="cog" value="0 0 0"/>
@@ -33,7 +33,7 @@
   assume NWU (otherwise cob is below cog?). 0.155
   -->
-  <xacro:property name="cob" value="0 0 0.05"/>
+  <xacro:property name="cob" value="0 0 0.15"/>
   <!-- Fluid density -->
-  <xacro:property name="rho" value="1000"/>
+  <xacro:property name="rho" value="1028"/>
   <!--
     Visual mesh file for the vehicle, usually in DAE (Collada) format. Be sure to store the
@@ -49,6 +49,5 @@
   <xacro:property name="use_simplified_mesh" value="false"/>
   <!-- Vehicle macro -->
-  <!-- <xacro:macro name="bluerov2_base" params="namespace debug *gazebo">  Mahya Changed to below-->
-  <!-- <xacro:macro name="bluerov2_base" params="namespace debug inertial_reference_frame"> -->
+  <!-- <xacro:macro name="bluerov2_base" params="namespace debug *gazebo"> -->
   <xacro:macro name="bluerov2_base" params="namespace *gazebo">
       <!-- Rigid body description of the base link -->
@@ -63,7 +62,7 @@
           <!-- <inertia ixx="525.39" ixy="1.44" ixz="33.41" iyy="794.20" iyz="2.6" izz="691.23"/> -->
           <inertia
-            ixx="0.7301" ixy="0.002048" ixz="0.003906"
-            iyy="0.7705" iyz="0.0018"
-            izz="0.8024" />
+            ixx="${0.2*mass*y_size*y_size + 0.2*mass*z_size*z_size}" ixy="0.0" ixz="0.0"
+            iyy="${0.2*mass*x_size*x_size + 0.2*mass*z_size*z_size}" iyz="0.0"
+            izz="${0.2*mass*x_size*x_size + 0.2*mass*y_size*y_size}" />
         </inertial>
         <!-- This visual geometry representation can be used when running

File: bluerov2_description/urdf/sensors_new.xacro (robot description, xacro)
@@ -21,4 +21,24 @@
     <origin xyz="0 0 0" rpy="0 0 0"/>
   </xacro:default_beacon> -->
+    <!-- Mount a GPS. -->
+  <xacro:default_gps namespace="${namespace}" parent_link="${namespace}/base_link" />
+  <!-- Mount a Pose 3D sensor. -->
+  <xacro:default_pose_3d_macro
+    namespace="${namespace}"
+    parent_link="${namespace}/base_link">
+    <!--   inertial_reference_frame="${inertial_reference_frame}"> -->
+   <origin xyz="0 0 0" rpy="0 0 0"/>
+    </xacro:default_pose_3d_macro>
+  <!-- Forward-looking sonar sensor -->
+  <xacro:forward_multibeam_p900 namespace="${namespace}" parent_link="${namespace}/base_link">
+    <origin xyz="0.0 0 -0.1" rpy="0 0 0"/>
+  </xacro:forward_multibeam_p900>
+  <!-- DVL  -->
+<xacro:default_dvl_macro
+  namespace="${namespace}"
+  parent_link="${namespace}/base_link">
+<!--   inertial_reference_frame="${inertial_reference_frame}"> -->
+  <origin xyz="0 0 0" rpy="0 ${0.5*pi} 0"/>
+</xacro:default_dvl_macro>
   <!-- Mount a camera -->
   <!-- <xacro:default_camera namespace="${namespace}" parent_link="${namespace}/base_link" suffix="front">
@@ -52,6 +72,5 @@
       <plugin filename="libgazebo_ros_range.so" name="gazebo_ros_range">
         <gaussianNoise>0.005</gaussianNoise>
-        <alwaysOn>1</alwaysOn>
-        <visualize>true</visualize>
+        <alwaysOn>true</alwaysOn>
         <updateRate>10</updateRate>
         <topicName>sonar</topicName>

File: bluerov2_description/urdf/sensors_original.xacro (robot description, xacro)
@@ -52,6 +52,5 @@
       <plugin filename="libgazebo_ros_range.so" name="gazebo_ros_range">
         <gaussianNoise>0.005</gaussianNoise>
-        <alwaysOn>1</alwaysOn>
-        <visualize>true</visualize>
+        <alwaysOn>true</alwaysOn>
         <updateRate>10</updateRate>
         <topicName>sonar</topicName>
